File: kicad/motors.kicad_sch (KiCad schematic)
At the start: 61 parts, among them J12 Conn_01x04_Pin, J3 Conn_01x04_Pin, J4 Conn_01x04_Pin, J5 Conn_01x04_Pin, J6 Conn_01x04_Pin, U3 DRV8825PWP, U4 DRV8825PWP, U5 DRV8825PWP, U6 TB67S109AFTG

Commit message: TB67S109A schematic wired
Parts:
- removed C1, C25: 100μF THT 36V, Capacitor_THT:C_Radial_D6.3mm_H11.0mm_P2.50mm, symbol Device:C_Polarized
- removed C11, C27: 1μF 0603 50V, Capacitor_SMD:C_0402_1005Metric, symbol Device:C
- removed D6: LED, LED_SMD:LED_0603_1608Metric, symbol Device:LED
- removed U3, U4, U5: DRV8825PWP, Package_SO:HTSSOP-28-1EP_4.4x9.7mm_P0.65mm_EP3.4x9.5mm_ThermalVias, symbol rephat-symbols:DRV8825PWP
- added C1, C25: 100 pF 0402 50V, Capacitor_SMD:C_0402_1005Metric, symbol Device:C
- added C11, C27: 100μF THT 36V, Capacitor_THT:C_Radial_D6.3mm_H11.0mm_P2.50mm, symbol Device:C_Polarized
- added C17: 0.1 μF 0402 50V, Capacitor_SMD:C_0402_1005Metric, symbol Device:C
- added C18: 0.1μF 0402 50V, Capacitor_SMD:C_0402_1005Metric, symbol Device:C
- added R26, R27, R30, R31, R35, R36: 100K 0402, Resistor_SMD:R_0402_1005Metric, symbol Device:R
- added R28, R29, R33, R34: 200m 2512 >2W 1%, Resistor_SMD:R_2512_6332Metric, symbol Device:R
- added R32: 20K 0402, Resistor_SMD:R_0402_1005Metric, symbol Device:R
- added U2, U3, U4: TB67S109AFTG, Package_DFN_QFN:QFN-48-1EP_7x7mm_P0.5mm_EP5.45x5.45mm_ThermalVias, symbol rephat-symbols:TB67S109AFTG
- C10, C26, C7: value 0.1μF 0402 50V -> 0.1 μF 0402 50V
- C12, C21, C28: value 0.1μF 0402 50V -> 1μF 0603 50V
- C20, C22, C24, C29: value 1μF 0603 50V -> 0.1μF 0402 50V
- C4: value 0.1μF 0402 50V -> 100 pF 0402 50V
- R13: value 200Ω 0402 -> 200m 2512 >2W 1%; footprint Resistor_SMD:R_0402_1005Metric -> Resistor_SMD:R_2512_6332Metric
- R14, R3: value R100 0603 -> 20K 0402; footprint Resistor_SMD:R_0603_1608Metric -> Resistor_SMD:R_0402_1005Metric
- R15, R16, R17: value R100 0603 -> 200m 2512 >2W 1%; footprint Resistor_SMD:R_0603_1608Metric -> Resistor_SMD:R_2512_6332Metric
- R18: value R100 0603 -> 100K 0402; footprint Resistor_SMD:R_0603_1608Metric -> Resistor_SMD:R_0402_1005Metric
Connections:
- net +3V3: no longer C20.1, C24.1, C29.1, RV1.1, RV2.1, RV3.1
- net +5V: now also C10.1, C26.1, C7.1, R11.2, R14.2, R18.1, R3.2, C17.1, R26.1, R32.2, R35.1, U2.34 (VCC), U3.34 (VCC), U4.34 (VCC); no longer R11.1
- net GND: now also C10.2, C23.2, C26.2, C30.2, C4.2, C7.2, C1.2, C11.2, C17.2, C18.2, C25.2, C27.2, R27.2, R30.2, R31.2, R36.2, U2.15 (GND), U2.18 (GND), U2.19 (GND), U2.22 (GND), U2.4 (RESET), U2.40 (GND), U2.5 (GND), U3.15 (GND), U3.18 (GND), U3.19 (GND), U3.22 (GND), U3.4 (RESET), U3.40 (GND), U3.5 (GND), U4.15 (GND), U4.18 (GND), U4.19 (GND), U4.22 (GND), U4.4 (RESET), U4.40 (GND), U4.5 (GND); no longer R14.2, R15.2, R16.2, R17.2, R18.2, R3.2, RV1.3, RV2.3, RV3.3
- net VCC: now also C23.1, C24.1, C30.1, R13.1, R15.1, R16.1, R17.1, C11.1, C27.1, R28.1, R29.1, R33.1, R34.1, U2.32 (VM), U3.32 (VM), U4.32 (VM); no longer C22.1, C23.2, C30.2, C7.2
- net at RN3.1 (R1.1): now also U4.3 (ENABLE)
- net at RN3.2 (R2.1): now also U4.44 (CW/CCW)
- net at RN3.3 (R3.1): now also U4.2 (CLK)
- net at C32.1, U6.43 (OSCM): now also R11.1; no longer R11.2
- net at JP2.2 (B): now also U3.46 (DMODE1)
- net at JP8.2 (B): now also U4.46 (DMODE1)
- net at J3.1 (Pin_1), J6.1 (Pin_1): now also U4.16 (OUTA-), U4.17 (OUTA-)
- net at J3.2 (Pin_2), J6.2 (Pin_2): now also U4.10 (OUTA+), U4.11 (OUTA+)
- net at J3.3 (Pin_3), J6.3 (Pin_3): now also U4.26 (OUTB+), U4.27 (OUTB+)
- net at J3.4 (Pin_4), J6.4 (Pin_4): now also U4.20 (OUTB-), U4.21 (OUTB-)
- net at JP5.2 (B): now also U2.46 (DMODE1)
- net Vref X: now reaches RV1.2
- net Vref X: now also C22.1, U3.41 (VREFB), U3.42 (VREFA)
- net at R14.1: now also C4.1, U3.43 (OSCM)
- net Vref Z: now reaches RV3.2
- net Vref Z: now also C29.1, U4.41 (VREFB), U4.42 (VREFA)
- net at JP9.2 (B): now also U4.47 (DMODE2)
- net at JP3.2 (B): now also U3.47 (DMODE2)
- net at RN1.1 (R1.1): now also U2.3 (ENABLE)
- net at RN1.2 (R2.1): now also U2.44 (CW/CCW)
- net at RN1.3 (R3.1): now also U2.2 (CLK)
- net at JP1.2 (B): now also U3.39 (DMODE0)
- net at J12.1 (Pin_1): now also U3.16 (OUTA-), U3.17 (OUTA-)
- net at J12.2 (Pin_2): now also U3.10 (OUTA+), U3.11 (OUTA+)
- net at J12.3 (Pin_3): now also U3.26 (OUTB+), U3.27 (OUTB+)
- net at J12.4 (Pin_4): now also U3.20 (OUTB-), U3.21 (OUTB-)
- net at U6.29 (RSB): now also U6.30 (RSB), R29.2
- net Vref A: now reaches U6.41 (VREFB)
- net Vref A: now also RV5.2, U6.42 (VREFA), C18.1
- net at U6.7 (RSA): now also U6.8 (RSA), R28.2
- net at RN2.1 (R1.1): now also U3.3 (ENABLE)
- net at RN2.2 (R2.1): now also U3.44 (CW/CCW)
- net at RN2.3 (R3.1): now also U3.2 (CLK)
- net at J4.1 (Pin_1): now also U2.16 (OUTA-), U2.17 (OUTA-)
- net at J4.2 (Pin_2): now also U2.10 (OUTA+), U2.11 (OUTA+)
- net at J4.3 (Pin_3): now also U2.26 (OUTB+), U2.27 (OUTB+)
- net at J4.4 (Pin_4): now also U2.20 (OUTB-), U2.21 (OUTB-)
- net at JP4.2 (B): now also U2.39 (DMODE0)
- net at R13.2: now also U2.7 (RSA), U2.8 (RSA)
- net at JP7.2 (B): now also U4.39 (DMODE0)
- net Vref Y: now reaches RV2.2
- net Vref Y: now also C20.1, U2.41 (VREFB), U2.42 (VREFA)
- net at JP6.2 (B): now also U2.47 (DMODE2)
- net at R3.1: now also C1.1, U2.43 (OSCM)
- net at RV5.1: now also R26.2
- net at RV5.3: now also R27.1
- new net: R30.1, RV2.3
- new net: R18.2, RV1.1
- new net: R31.1, RV1.3
- new net: R34.2, U4.29 (RSB), U4.30 (RSB)
- new net: C25.1, R32.1, U4.43 (OSCM)
- new net: R33.2, U4.7 (RSA), U4.8 (RSA)
- new net: R17.2, U3.29 (RSB), U3.30 (RSB)
- new net: R15.2, U3.7 (RSA), U3.8 (RSA)
- new net: R19.2, RV2.1
- new net: R36.1, RV3.3
- new net: R35.2, RV3.1
- new net: R16.2, U2.29 (RSB), U2.30 (RSB)
- now unconnected: U6.38 (LO)
- no-connect marks 27 -> 16
Other:
- moved on the sheet: C31, C32, C33, C34, J12, J3, J4, J5, J6, JP10, JP11, JP12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

Commit message: cleanup
Parts:
- R18, R19, R26, R35: value 100K 0402 -> 8K2 0402
- R27, R30, R31, R36: value 100K 0402 -> 2K7 0402
Changed lines of the file:
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@@
 			)
 		)
-		(property "Value" "100K 0402"
+		(property "Value" "2K7 0402"
 			(at 353.06 101.6 0)
 			(effects
@@
 			)
 		)
-		(property "Value" "100K 0402"
+		(property "Value" "2K7 0402"
 			(at 157.48 104.14 0)
 			(effects
@@
 			)
 		)
-		(property "Value" "100K 0402"
+		(property "Value" "2K7 0402"
 			(at 354.33 214.63 0)
 			(effects
@@
 			)
 		)
-		(property "Value" "100K 0402"
+		(property "Value" "2K7 0402"
 			(at 160.02 232.41 0)
 			(effects
@@
 			)
 		)
-		(property "Value" "100K 0402"
+		(property "Value" "8K2 0402"
 			(at 157.48 83.82 0)
 			(effects
@@
 			)
 		)
-		(property "Value" "100K 0402"
+		(property "Value" "8K2 0402"
 			(at 354.33 194.31 0)
 			(effects
@@
 			)
 		)
-		(property "Value" "100K 0402"
+		(property "Value" "8K2 0402"
 			(at 160.02 212.09 0)
 			(effects
@@
 			)
 		)
-		(property "Value" "100K 0402"
+		(property "Value" "8K2 0402"
 			(at 353.06 81.28 0)
 			(effects
