File: kicad/RepHat.kicad_pcb (KiCad board)
At the start: 2 copper layers, 65 x 56 mm, 42 parts, among them J1 GPIO, J10 Conn_01x04_Pin, J11 Conn_01x04_Pin, J12 Conn_01x03_Pin, J13 Conn_01x03_Pin, J14 Conn_01x03_Pin, J15 Conn_01x03_Pin, J16 Conn_01x03_Pin, J17 Screw_Terminal_01x02, J2 Screw_Terminal_01x02, J3 Conn_02x03_Odd_Even, J4 Conn_01x04_Pin, J5 Conn_02x03_Odd_Even, J6 Conn_01x04_Pin, J7 Conn_02x03_Odd_Even, J8 Conn_01x04_Pin, J9 Conn_02x03_Odd_Even, U1 LMR51450FNDRRR

Commit message: Miniaturizing the stepper drivers. They're still too big
Parts:
- removed A1, A2, A3, A4: Pololu_Breakout_A4988, Module:Pololu_Breakout-16_15.2x20.3mm
- removed J10, J11, J8: Conn_01x04_Pin, Connector_JST:JST_XH_B4B-XH-A_1x04_P2.50mm_Vertical
- removed J14, J15, J16: Conn_01x03_Pin, Connector_JST:JST_XH_B3B-XH-A_1x03_P2.50mm_Vertical
- removed J7, J9: Conn_02x03_Odd_Even, Connector_PinHeader_2.54mm:PinHeader_2x03_P2.54mm_Vertical
- added ASTOP1: Conn_01x03_Pin, Connector_JST:JST_XH_B3B-XH-A_1x03_P2.50mm_Vertical, F.Cu at (108.2, 67.0)
- added C13: 0.1uF, Capacitor_SMD:C_0402_1005Metric, F.Cu at (117.5, 86.9)
- added C14: 0.1uF, Capacitor_SMD:C_0402_1005Metric, F.Cu at (115.5, 81.7)
- added C15: 0.1uF, Capacitor_SMD:C_0402_1005Metric, F.Cu at (115.6, 74.6)
- added C16: 0.1uF, Capacitor_SMD:C_0402_1005Metric, F.Cu at (115.2, 67.0)
- added C17: 1 uF, Capacitor_SMD:C_0402_1005Metric, F.Cu at (103.5, 56.7)
- added C18: 0.1uF, Capacitor_SMD:C_0402_1005Metric, F.Cu at (103.5, 55.1)
- added C19: 100 uF, Capacitor_THT:C_Radial_D6.3mm_H11.0mm_P2.50mm, F.Cu at (-6.34, 177.3)
- added C20: 0.1 uF, Capacitor_SMD:C_0402_1005Metric, F.Cu at (2.89, 147.7)
- added C21: 0.1 uF, Capacitor_SMD:C_0402_1005Metric, F.Cu at (2.89, 150.2)
- added C22: 1 uF, Capacitor_SMD:C_0402_1005Metric, F.Cu at (-10.7, 177.6)
- added C23: 0.1 uF, Capacitor_SMD:C_0402_1005Metric, F.Cu at (2.89, 152.7)
- added C24: 22 nF 50V, Capacitor_SMD:C_0402_1005Metric, F.Cu at (2.89, 155.2)
- added C25: 0.1 uF, Capacitor_SMD:C_0402_1005Metric, F.Cu at (2.89, 157.7)
- added C26: 0.1 uF, Capacitor_SMD:C_0402_1005Metric, F.Cu at (232.5, 160.2)
- added C27: 0.1 uF, Capacitor_SMD:C_0402_1005Metric, F.Cu at (232.5, 162.7)
- added C28: 0.1 uF, Capacitor_SMD:C_0402_1005Metric, F.Cu at (236.5, 142.6)
- added C29: 0.1 uF, Capacitor_SMD:C_0402_1005Metric, F.Cu at (123.5, 140.4)
- added C30: 1 uF, Capacitor_SMD:C_0402_1005Metric, F.Cu at (105.9, 176.2)
- added C31: 100 uF, Capacitor_THT:C_Radial_D6.3mm_H11.0mm_P2.50mm, F.Cu at (110.3, 175.7)
- added C32: 22 nF 50V, Capacitor_SMD:C_0402_1005Metric, F.Cu at (123.5, 142.9)
- added C33: 0.1 uF, Capacitor_SMD:C_0402_1005Metric, F.Cu at (123.5, 145.4)
- added C34: 0.1 uF, Capacitor_SMD:C_0402_1005Metric, F.Cu at (123.5, 147.9)
- added C35: 0.1 uF, Capacitor_SMD:C_0402_1005Metric, F.Cu at (123.5, 150.5)
- added C36: 0.1 uF, Capacitor_SMD:C_0402_1005Metric, F.Cu at (335.0, 158.9)
- added C37: 1 uF, Capacitor_SMD:C_0402_1005Metric, F.Cu at (317.4, 185.5)
- added C38: 100 uF, Capacitor_THT:C_Radial_D6.3mm_H11.0mm_P2.50mm, F.Cu at (321.8, 184.8)
- added C39: 22 nF 50V, Capacitor_SMD:C_0402_1005Metric, F.Cu at (335.0, 161.4)
- added C40: 0.1 uF, Capacitor_SMD:C_0402_1005Metric, F.Cu at (335.0, 164.0)
- added C41: 0.1 uF, Capacitor_SMD:C_0402_1005Metric, F.Cu at (339.0, 143.9)
- added C42: 0.1 uF, Capacitor_SMD:C_0402_1005Metric, F.Cu at (339.0, 146.4)
- added JP1: SPREADCYCLE, Jumper:SolderJumper-2_P1.3mm_Bridged_RoundedPad1.0x1.5mm, F.Cu at (3.06, 165.8)
- added JP10: MS1, Jumper:SolderJumper-2_P1.3mm_Bridged_RoundedPad1.0x1.5mm, F.Cu at (344.2, 167.0)
- added JP11: MS2, Jumper:SolderJumper-2_P1.3mm_Bridged_RoundedPad1.0x1.5mm, F.Cu at (344.2, 170.5)
- added JP12: SPREADCYCLE, Jumper:SolderJumper-2_P1.3mm_Bridged_RoundedPad1.0x1.5mm, F.Cu at (344.2, 174.1)
- added JP2: MS1, Jumper:SolderJumper-2_P1.3mm_Bridged_RoundedPad1.0x1.5mm, F.Cu at (3.06, 169.3)
- added JP3: MS2, Jumper:SolderJumper-2_P1.3mm_Bridged_RoundedPad1.0x1.5mm, F.Cu at (3.06, 172.9)
- added JP4: MS1, Jumper:SolderJumper-2_P1.3mm_Bridged_RoundedPad1.0x1.5mm, F.Cu at (237.0, 165.8)
- added JP5: MS2, Jumper:SolderJumper-2_P1.3mm_Bridged_RoundedPad1.0x1.5mm, F.Cu at (237.0, 169.3)
- added JP6: SPREADCYCLE, Jumper:SolderJumper-2_P1.3mm_Bridged_RoundedPad1.0x1.5mm, F.Cu at (237.0, 172.9)
- added JP7: MS1, Jumper:SolderJumper-2_P1.3mm_Bridged_RoundedPad1.0x1.5mm, F.Cu at (128.4, 161.0)
- added JP8: MS2, Jumper:SolderJumper-2_P1.3mm_Bridged_RoundedPad1.0x1.5mm, F.Cu at (128.4, 164.6)
- added JP9: SPREADCYCLE, Jumper:SolderJumper-2_P1.3mm_Bridged_RoundedPad1.0x1.5mm, F.Cu at (128.4, 168.1)
- added R10: 100 R, Resistor_SMD:R_0402_1005Metric, F.Cu at (125.5, 86.9)
- added R11: 100 R, Resistor_SMD:R_0402_1005Metric, F.Cu at (126.1, 79.6)
- added R12: 100 R, Resistor_SMD:R_0402_1005Metric, F.Cu at (117.8, 74.6)
- added R13: 100 R, Resistor_SMD:R_0402_1005Metric, F.Cu at (114.2, 65.0)
- added R14: 110 mR, Resistor_SMD:R_2010_5025Metric, F.Cu at (10.9, 147.7)
- added R15: 110 mR, Resistor_SMD:R_2010_5025Metric, F.Cu at (10.9, 150.2)
- added R16: 100 K, Resistor_SMD:R_0402_1005Metric, F.Cu at (10.9, 152.7)
- added R17: 100 K, Resistor_SMD:R_0402_1005Metric, F.Cu at (240.5, 155.2)
- added R18: 110 mR, Resistor_SMD:R_2010_5025Metric, F.Cu at (240.5, 157.7)
- added R19: 110 mR, Resistor_SMD:R_2010_5025Metric, F.Cu at (240.5, 160.2)
- added R20: 100 K, Resistor_SMD:R_0402_1005Metric, F.Cu at (127.5, 158.0)
- added R21: 110 mR, Resistor_SMD:R_2010_5025Metric, F.Cu at (131.5, 137.9)
- added R22: 110 mR, Resistor_SMD:R_2010_5025Metric, F.Cu at (131.5, 140.4)
- added R23: 100 K, Resistor_SMD:R_0402_1005Metric, F.Cu at (343.0, 148.9)
- added R24: 110 mR, Resistor_SMD:R_2010_5025Metric, F.Cu at (343.0, 151.4)
- added R25: 110 mR, Resistor_SMD:R_2010_5025Metric, F.Cu at (343.0, 153.9)
- added R26: 100 R, Resistor_SMD:R_0402_1005Metric, F.Cu at (10.8, 188.4)
- added R27: 100 R, Resistor_SMD:R_0402_1005Metric, F.Cu at (10.8, 190.9)
- added R28: 100 R, Resistor_SMD:R_0402_1005Metric, F.Cu at (10.8, 193.4)
- added R29: 100 R, Resistor_SMD:R_0402_1005Metric, F.Cu at (127.4, 191.2)
- added R30: 100 R, Resistor_SMD:R_0402_1005Metric, F.Cu at (131.4, 183.6)
- added R31: 100 R, Resistor_SMD:R_0402_1005Metric, F.Cu at (131.4, 186.1)
- added R32: 100 R, Resistor_SMD:R_0402_1005Metric, F.Cu at (342.9, 194.6)
- added R33: 100 R, Resistor_SMD:R_0402_1005Metric, F.Cu at (342.9, 197.1)
- added R34: 100 R, Resistor_SMD:R_0402_1005Metric, F.Cu at (346.9, 189.6)
- added R35: 100 R, Resistor_SMD:R_0402_1005Metric, F.Cu at (248.4, 190.9)
- added R36: 100 R, Resistor_SMD:R_0402_1005Metric, F.Cu at (248.4, 193.4)
- added R37: 100 R, Resistor_SMD:R_0402_1005Metric, F.Cu at (248.4, 195.9)
- added R4: 100 kR, Resistor_SMD:R_0402_1005Metric, F.Cu at (28.4, 83.1)
- added R5: 14.7 kR, Resistor_SMD:R_0402_1005Metric, F.Cu at (28.4, 85.6)
- added R6: 100 K, Resistor_SMD:R_0402_1005Metric, F.Cu at (121.5, 89.4)
- added R7: 100 K, Resistor_SMD:R_0402_1005Metric, F.Cu at (113.8, 81.6)
- added R8: 100 K, Resistor_SMD:R_0402_1005Metric, F.Cu at (114.0, 74.8)
- added R9: 100 K, Resistor_SMD:R_0402_1005Metric, F.Cu at (114.2, 67.0)
- added RV1: 100K, Potentiometer_SMD:Potentiometer_Bourns_TC33X_Vertical, F.Cu at (20.1, 143.8)
- added RV2: 100K, Potentiometer_SMD:Potentiometer_Bourns_TC33X_Vertical, F.Cu at (249.7, 148.5)
- added RV3: 100K, Potentiometer_SMD:Potentiometer_Bourns_TC33X_Vertical, F.Cu at (136.7, 148.5)
- added RV4: 100K, Potentiometer_SMD:Potentiometer_Bourns_TC33X_Vertical, F.Cu at (348.2, 159.2)
- added U2: SN74LVC07APW, Package_SO:TSSOP-14-1EP_4.4x5mm_P0.65mm, F.Cu at (108.3, 58.1)
- added U3: TMC2209-LA, rephat-parts:QFN28_5X5_TRI-M, F.Cu at (19.2, 163.5)
- added U4: TMC2209-LA, rephat-parts:QFN28_5X5_TRI-M, F.Cu at (212.1, 153.4)
- added U5: TMC2209-LA, rephat-parts:QFN28_5X5_TRI-M, F.Cu at (99.1, 156.6)
- added U6: TMC2209-LA, rephat-parts:QFN28_5X5_TRI-M, F.Cu at (310.5, 170.6)
- added XSTOP1: Conn_01x03_Pin, Connector_JST:JST_XH_B3B-XH-A_1x03_P2.50mm_Vertical, F.Cu at (108.2, 88.0)
- added YSTOP1: Conn_01x03_Pin, Connector_JST:JST_XH_B3B-XH-A_1x03_P2.50mm_Vertical, F.Cu at (108.2, 81.0)
- added ZSTOP1: Conn_01x03_Pin, Connector_JST:JST_XH_B3B-XH-A_1x03_P2.50mm_Vertical, F.Cu at (108.2, 74.0)
- C1: value 100 uF -> 0.1 uF; footprint Capacitor_THT:C_Disc_D3.0mm_W1.6mm_P2.50mm -> Capacitor_SMD:C_0402_1005Metric
- C10: value 100 uF -> 1 uF; footprint Capacitor_THT:C_Disc_D3.0mm_W1.6mm_P2.50mm -> Capacitor_SMD:C_0402_1005Metric
- C11: footprint Capacitor_THT:C_Disc_D3.0mm_W1.6mm_P2.50mm -> Capacitor_THT:C_Radial_D6.3mm_H11.0mm_P2.50mm
- C12: value 100 uF -> 22 nF 50V; footprint Capacitor_THT:C_Disc_D3.0mm_W1.6mm_P2.50mm -> Capacitor_SMD:C_0402_1005Metric
- C2, C5, C6, C7: footprint Capacitor_SMD:C_0603_1608Metric -> Capacitor_SMD:C_0402_1005Metric
- C3: value 10 uF -> 1 uF; footprint Capacitor_SMD:C_0603_1608Metric -> Capacitor_SMD:C_0402_1005Metric
- C4: value 1 uF -> 47 uF; footprint Capacitor_SMD:C_0603_1608Metric -> Capacitor_SMD:C_1206_3216Metric
- J12: value Conn_01x03_Pin -> Conn_01x04_Pin; footprint Connector_JST:JST_XH_B3B-XH-A_1x03_P2.50mm_Vertical -> Connector_JST:JST_XH_B4B-XH-A_1x04_P2.50mm_Vertical
- J13: footprint Connector_JST:JST_XH_B3B-XH-A_1x03_P2.50mm_Vertical -> Connector_PinHeader_2.54mm:PinHeader_1x03_P2.54mm_Vertical
- J17, J2: footprint TerminalBlock_WAGO:TerminalBlock_WAGO_236-102_1x02_P5.00mm_45Degree -> TerminalBlock:TerminalBlock_bornier-2_P5.08mm
- J3, J5: value Conn_02x03_Odd_Even -> Conn_01x04_Pin; footprint Connector_PinHeader_2.54mm:PinHeader_2x03_P2.54mm_Vertical -> Connector_JST:JST_XH_B4B-XH-A_1x04_P2.50mm_Vertical
- L1: value 5.6 uH -> 3.3 uH
- R1, R2, R3: footprint Resistor_SMD:R_0603_1608Metric -> Resistor_SMD:R_0402_1005Metric
- moved C2 142.5 mm to (24.4, 75.5)
- moved C3 142.5 mm to (24.4, 78.0)
- moved C5 141.3 mm to (24.4, 80.5)
- moved C6 141.3 mm to (24.4, 83.1)
- moved C7 141.3 mm to (24.4, 85.6)
- moved L1 141.0 mm to (29.8, 68.4)
- moved C1 136.1 mm to (232.5, 142.6)
- moved C8 135.1 mm to (33.3, 79.3)
- moved C9 135.1 mm to (33.3, 82.6)
- moved U1 133.7 mm to (39.2, 76.7)
- moved C4 132.5 mm to (33.3, 75.9)
- moved R1 132.3 mm to (28.4, 75.5)
- moved R2 132.3 mm to (28.4, 78.0)
- moved R3 132.3 mm to (28.4, 80.5)
- moved C10 130.4 mm to (218.9, 174.3)
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Connections:
- C1 pad 1: VCC -> Net-(U4-5VOUT)
- C10 pad 1: VCC -> +3.3V
- C12 pad 1: VCC -> Net-(U4-CPI)
- C12 pad 2: GND -> Net-(U4-CPO)
- C7 pad 2: Net-(U1-FB) -> GND
- J12 pad 1: /GPIO19/PCM.FS -> Net-(J12-Pin_1)
- J12 pad 2: GND -> Net-(J12-Pin_2)
- J12 pad 3: +3.3V -> Net-(J12-Pin_3)
- J3 pad 1: +3.3V -> Net-(J3-Pin_1)
- J3 pad 2: Net-(A1-MS1) -> Net-(J3-Pin_2)
- J3 pad 3: +3.3V -> Net-(J3-Pin_3)
- J3 pad 4: Net-(A1-MS2) -> Net-(J3-Pin_4)
- J5 pad 1: +3.3V -> Net-(J5-Pin_1)
- J5 pad 3: +3.3V -> Net-(J5-Pin_3)
- J6 pad 1: Net-(A2-2B) -> Net-(J3-Pin_1)
- J6 pad 2: Net-(A2-2A) -> Net-(J3-Pin_2)
- J6 pad 3: Net-(A2-1A) -> Net-(J3-Pin_3)
- J6 pad 4: Net-(A2-1B) -> Net-(J3-Pin_4)
- R1 pad 1: GND -> Net-(U1-FB)
- R1 pad 2: Net-(U1-FB) -> GND
- U1 pad 5: GND -> Net-(U1-PG)
- U1 pad 6: unconnected-(U1-RT-Pad6) -> Net-(U1-RT)
Other:
- board text added: "+5V GND PIN"

Commit message: PCB redo
Parts:
- removed C37: 1 uF, Capacitor_SMD:C_0402_1005Metric
- removed C38: 100 uF, Capacitor_THT:C_Radial_D6.3mm_H11.0mm_P2.50mm
- removed C39: 22 nF 50V, Capacitor_SMD:C_0402_1005Metric
- removed C41, C42: 0.1 uF, Capacitor_SMD:C_0402_1005Metric
- removed R21, R22: 110 mR, Resistor_SMD:R_2010_5025Metric
- removed R23: 100 K, Resistor_SMD:R_0402_1005Metric
- removed R26, R27, R28, R29, R30, R31, R32, R33, R34, R35, R36, R37: 100 R, Resistor_SMD:R_0402_1005Metric
- added D1: SMBJ5.0A, Diode_SMD:D_SMA-SMB_Universal_Handsoldering, F.Cu at (115.1, 159.1)
- added D2: BAV99S, Package_TO_SOT_SMD:SOT-363_SC-70-6, F.Cu at (162.0, 133.8)
- added D3: BAV99S, Package_TO_SOT_SMD:SOT-363_SC-70-6, F.Cu at (162.0, 137.8)
- added Q1: DMG2301L, Package_TO_SOT_SMD:SOT-23, F.Cu at (116.7, 172.2)
- added Q2: DMMT5401, Package_TO_SOT_SMD:SOT-23-6, F.Cu at (116.8, 167.6)
- C1, C25: value 0.1 uF -> 100μF THT 36V; footprint Capacitor_SMD:C_0402_1005Metric -> Capacitor_THT:C_Radial_D6.3mm_H11.0mm_P2.50mm
- C10, C17, C30: value 1 uF -> 0.1μF 0402 50V
- C11: value 100 uF -> 1μF 0603 50V; footprint Capacitor_THT:C_Radial_D6.3mm_H11.0mm_P2.50mm -> Capacitor_SMD:C_0402_1005Metric
- C12, C32: value 22 nF 50V -> 0.1μF 0402 50V
- C13, C14, C15, C16, C18, C5: value 0.1uF -> 0.1μF 0402 50V
- C19, C31: value 100 uF -> 100μF THT 36V
- C2: value 10 uF -> 10μF 0402 16V
- C20, C27, C29, C33, C35: value 0.1 uF -> 1μF 0603 50V
- C21, C23, C26, C28, C34, C36: value 0.1 uF -> 0.1μF 0402 50V
- C22, C3: value 1 uF -> 1μF 0603 50V
- C24: value 22 nF 50V -> 1μF 0603 50V
- C4: value 47 uF -> 0.1μF 0402 50V; footprint Capacitor_SMD:C_1206_3216Metric -> Capacitor_SMD:C_0402_1005Metric
- C40: value 0.1 uF -> 47uF 1206 10V; footprint Capacitor_SMD:C_0402_1005Metric -> Capacitor_SMD:C_1206_3216Metric
- C6: value 0.1 uF -> 0.1μF 0402 16V
- C7: value 33 pF -> 0.1μF 0402 50V
- C8, C9: value 47 uF -> 47uF 1206 10V
- JP1, JP12, JP6, JP9: value SPREADCYCLE -> CFG
- JP10, JP2, JP4, JP7: value MS1 -> CFG
- JP11, JP3, JP5, JP8: value MS2 -> CFG
- R1: value 19.1 kR -> 19k1 0402
- R10, R11, R12, R13: value 100 R -> 10K 0402
- R14, R15, R18, R19: value 110 mR -> R110 2010 0.7W Film
- R16, R17, R20: value 100 K -> R110 2010 0.7W Film; footprint Resistor_SMD:R_0402_1005Metric -> Resistor_SMD:R_2010_5025Metric
- R2: value 100 kR -> 1pF 0402
- R24: value 110 mR -> 10K 0402; footprint Resistor_SMD:R_2010_5025Metric -> Resistor_SMD:R_0402_1005Metric
- R25: value 110 mR -> 47K 0402; footprint Resistor_SMD:R_2010_5025Metric -> Resistor_SMD:R_0402_1005Metric
- R3: value 1 kR -> R110 2010 0.7W Film; footprint Resistor_SMD:R_0402_1005Metric -> Resistor_SMD:R_2010_5025Metric
- R4: value 100 kR -> 100k 0402
- R5: value 14.7 kR -> 14k7 0402
- R6, R7, R8, R9: value 100 K -> 100K 0402
- U3, U4, U5, U6: value TMC2209-LA -> DRV8825PWP; footprint rephat-parts:QFN28_5X5_TRI-M -> Package_SO:HTSSOP-28-1EP_4.4x9.7mm_P0.65mm_EP3.4x9.5mm_ThermalVias
- moved R24 232.9 mm to (111.0, 172.5)
- moved R25 232.9 mm to (111.0, 174.5)
- moved C40 217.9 mm to (117.1, 163.5)
- moved RV4 217.6 mm to (130.9, 147.9)
- moved JP10 206.1 mm to (143.0, 122.4)
- moved JP11 206.1 mm to (143.0, 125.9)
- moved JP12 206.1 mm to (143.0, 129.5)
- moved C36 192.0 mm to (143.9, 140.1)
- moved U6 177.8 mm to (141.7, 114.9)
- moved C22 154.6 mm to (138.2, 136.2)
- moved R1 151.6 mm to (164.0, 143.4)
- moved R2 151.4 mm to (164.0, 145.4)
- moved R4 150.1 mm to (164.0, 147.4)
- moved R5 149.8 mm to (164.0, 149.4)
- moved L1 148.7 mm to (155.2, 148.3)
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Connections:
- ASTOP1 pad 1: Net-(ASTOP1-Pin_1) -> /Endstops/Stop A
- C1 pad 1: Net-(U4-5VOUT) -> VCC
- C10 pad 1: +3.3V -> Net-(U4-CP2)
- C10 pad 2: GND -> Net-(U4-CP1)
- C12 pad 1: Net-(U4-CPI) -> VCC
- C12 pad 2: Net-(U4-CPO) -> GND
- C13 pad 1: Net-(XSTOP1-Pin_1) -> /Endstops/Stop X
- C14 pad 1: Net-(YSTOP1-Pin_1) -> /Endstops/Stop Y
- C15 pad 1: Net-(ZSTOP1-Pin_1) -> /Endstops/Stop Z
- C16 pad 1: Net-(ASTOP1-Pin_1) -> /Endstops/Stop A
- C20 pad 1: VCC -> +3V3
- C22 pad 1: +3.3V -> VCC
- C23 pad 1: Net-(U3-5VOUT) -> Net-(U4-VCP)
- C23 pad 2: GND -> VCC
- C24 pad 1: Net-(U3-CPI) -> +3V3
- C24 pad 2: Net-(U3-CPO) -> GND
- C25 pad 2: Net-(U3-VCP) -> GND
- C26 pad 1: VCC -> Net-(U5-CP2)
- C26 pad 2: GND -> Net-(U5-CP1)
- C27 pad 2: Net-(U4-VCP) -> GND
- C29 pad 1: Net-(U5-5VOUT) -> +3V3
- C30 pad 1: +3.3V -> Net-(U5-VCP)
- C30 pad 2: GND -> VCC
- C32 pad 1: Net-(U5-CPI) -> Net-(U6-CP2)
- C32 pad 2: Net-(U5-CPO) -> Net-(U6-CP1)
- C34 pad 2: Net-(U5-VCP) -> GND
- C35 pad 1: VCC -> +3V3
- C36 pad 1: Net-(U6-5VOUT) -> Net-(U6-VCP)
- C36 pad 2: GND -> VCC
- C4 pad 1: VCC -> Net-(U3-CP2)
- C4 pad 2: GND -> Net-(U3-CP1)
- C40 pad 1: VCC -> Net-(D1-A)
- C7 pad 1: Net-(C7-Pad1) -> Net-(U3-VCP)
- C7 pad 2: GND -> VCC
- J1 pad 2: +5V -> Net-(D1-A)
- J1 pad 4: +5V -> Net-(D1-A)
- JP1 pad 1: GND -> +3V3
- JP10 pad 1: +3.3V -> +3V3
- JP11 pad 1: +3.3V -> +3V3
- JP12 pad 1: GND -> +3V3
- JP2 pad 1: +3.3V -> +3V3
- JP3 pad 1: +3.3V -> +3V3
- JP4 pad 1: +3.3V -> +3V3
- JP5 pad 1: +3.3V -> +3V3
- JP6 pad 1: GND -> +3V3
- JP7 pad 1: +3.3V -> +3V3
- JP8 pad 1: +3.3V -> +3V3
- JP9 pad 1: GND -> +3V3
- R10 pad 1: Net-(XSTOP1-Pin_1) -> /Endstops/Stop X
- R10 pad 2: /Endstops/Stop X -> Net-(D2A-K3A4)
- R11 pad 1: Net-(YSTOP1-Pin_1) -> /Endstops/Stop Y
- R11 pad 2: /Endstops/Stop Y -> Net-(D2B-K1A2)
- R12 pad 1: Net-(ZSTOP1-Pin_1) -> /Endstops/Stop Z
- R12 pad 2: /Endstops/Stop Z -> Net-(D3A-K3A4)
- R13 pad 1: Net-(ASTOP1-Pin_1) -> /Endstops/Stop A
- R13 pad 2: /Endstops/Stop A -> Net-(D3B-K1A2)
- R14 pad 1: Net-(U3-BRB) -> Net-(U3-ISENB)
- R15 pad 1: Net-(U3-BRA) -> Net-(U3-ISENA)
- R16 pad 1: Net-(U3-5VOUT) -> Net-(U4-ISENA)
- R16 pad 2: Net-(R16-Pad2) -> GND
- R17 pad 1: Net-(U4-5VOUT) -> Net-(U5-ISENB)
- R17 pad 2: Net-(R17-Pad2) -> GND
- R18 pad 1: Net-(U4-BRB) -> Net-(U5-ISENA)
- R19 pad 1: Net-(U4-BRA) -> Net-(U6-ISENB)
- R20 pad 1: Net-(U5-5VOUT) -> Net-(U6-ISENA)
- R20 pad 2: Net-(R20-Pad2) -> GND
- R24 pad 1: Net-(U6-BRB) -> Net-(Q2A-B1)
- R25 pad 1: Net-(U6-BRA) -> Net-(Q1-G)
- R3 pad 1: +5V -> Net-(U4-ISENB)
- R3 pad 2: Net-(C7-Pad1) -> GND
- R6 pad 1: Net-(XSTOP1-Pin_1) -> /Endstops/Stop X
- R7 pad 1: Net-(YSTOP1-Pin_1) -> /Endstops/Stop Y
- R8 pad 1: Net-(ZSTOP1-Pin_1) -> /Endstops/Stop Z
- R9 pad 1: Net-(ASTOP1-Pin_1) -> /Endstops/Stop A
- RV1 pad 1: GND -> +3V3
- RV1 pad 2: Net-(U3-VREF) -> Net-(U3-AVREF)
- RV1 pad 3: Net-(R16-Pad2) -> GND
- RV2 pad 1: GND -> +3V3
- RV2 pad 2: Net-(U4-VREF) -> Net-(U4-AVREF)
- RV2 pad 3: Net-(R17-Pad2) -> GND
- RV3 pad 1: GND -> +3V3
- RV3 pad 2: Net-(U5-VREF) -> Net-(U5-AVREF)
- RV3 pad 3: Net-(R20-Pad2) -> GND
- RV4 pad 1: GND -> +3V3
- RV4 pad 2: Net-(U6-VREF) -> Net-(U6-AVREF)
- RV4 pad 3: Net-(R23-Pad2) -> GND
- U3 pad 1: Net-(J12-Pin_4) -> Net-(U3-CP1)
- U3 pad 10: Net-(JP3-B) -> Net-(J12-Pin_3)
- U3 pad 11: unconnected-(U3-DIAG-Pad11) -> VCC
- U3 pad 12: unconnected-(U3-INDEX-Pad12) -> Net-(U3-AVREF)
- U3 pad 13: GND -> Net-(U3-AVREF)
- U3 pad 14: +3.3V -> GND
- U3 pad 15: +3.3V -> +3V3
- U3 pad 16: Net-(U3-STEP) -> unconnected-(U3-NRESET-Pad16)
- U3 pad 17: Net-(U3-VREF) -> unconnected-(U3-NSLEEP-Pad17)
- U3 pad 18: GND -> unconnected-(U3-NFAULT-Pad18)
- U3 pad 19: Net-(U3-DIR) -> unconnected-(U3-DECAY-Pad19)
- U3 pad 2: Net-(U3-ENN) -> Net-(U3-CP2)
- U3 pad 20: GND -> /GPIO3/SCL1
- U3 pad 21: Net-(J12-Pin_1) -> /GPIO4/GPCLK0
- U3 pad 22: VCC -> /GPIO2/SDA1
- U3 pad 23: Net-(U3-BRA) -> unconnected-(U3-NC-Pad23)
- U3 pad 24: Net-(J12-Pin_2) -> Net-(JP1-B)
- U3 pad 25: unconnected-(U3-NC-Pad25) -> Net-(JP2-B)
- U3 pad 26: Net-(J12-Pin_3) -> Net-(JP3-B)
- U3 pad 27: Net-(U3-BRB) -> unconnected-(U3-NHOME-Pad27)
- U3 pad 28: VCC -> GND
- U3 pad 3: GND -> Net-(U3-VCP)
- U3 pad 4: Net-(U3-CPO) -> VCC
- U3 pad 5: Net-(U3-CPI) -> Net-(J12-Pin_2)
- U3 pad 6: Net-(U3-VCP) -> Net-(U3-ISENA)
- U3 pad 7: Net-(JP1-B) -> Net-(J12-Pin_1)
- U3 pad 8: Net-(U3-5VOUT) -> Net-(J12-Pin_4)
- U3 pad 9: Net-(JP2-B) -> Net-(U3-ISENB)
- U4 pad 1: Net-(J3-Pin_4) -> Net-(U4-CP1)
- U4 pad 10: Net-(JP5-B) -> Net-(J4-Pin_3)
- U4 pad 11: unconnected-(U4-DIAG-Pad11) -> VCC
- U4 pad 12: unconnected-(U4-INDEX-Pad12) -> Net-(U4-AVREF)
- U4 pad 13: GND -> Net-(U4-AVREF)
- U4 pad 14: +3.3V -> GND
- U4 pad 15: +3.3V -> +3V3
- U4 pad 16: Net-(U4-STEP) -> unconnected-(U4-NRESET-Pad16)
- U4 pad 17: Net-(U4-VREF) -> unconnected-(U4-NSLEEP-Pad17)
- U4 pad 18: GND -> unconnected-(U4-NFAULT-Pad18)
- U4 pad 19: Net-(U4-DIR) -> unconnected-(U4-DECAY-Pad19)
- U4 pad 2: Net-(U4-ENN) -> Net-(U4-CP2)
- U4 pad 20: GND -> /GPIO27
- U4 pad 21: Net-(J3-Pin_1) -> /GPIO17
- U4 pad 22: VCC -> /GPIO22
- U4 pad 23: Net-(U4-BRA) -> unconnected-(U4-NC-Pad23)
- U4 pad 24: Net-(J3-Pin_2) -> Net-(JP4-B)
- U4 pad 25: unconnected-(U4-NC-Pad25) -> Net-(JP5-B)
- U4 pad 26: Net-(J3-Pin_3) -> Net-(JP6-B)
- U4 pad 27: Net-(U4-BRB) -> unconnected-(U4-NHOME-Pad27)
- U4 pad 28: VCC -> GND
- U4 pad 3: GND -> Net-(U4-VCP)
- U4 pad 4: Net-(U4-CPO) -> VCC
- U4 pad 5: Net-(U4-CPI) -> Net-(J4-Pin_2)
- U4 pad 6: Net-(U4-VCP) -> Net-(U4-ISENA)
- U4 pad 7: Net-(JP6-B) -> Net-(J4-Pin_1)
- U4 pad 8: Net-(U4-5VOUT) -> Net-(J4-Pin_4)
- U4 pad 9: Net-(JP4-B) -> Net-(U4-ISENB)
- U5 pad 1: Net-(J4-Pin_4) -> Net-(U5-CP1)
- U5 pad 10: Net-(JP8-B) -> Net-(J3-Pin_3)
- U5 pad 11: unconnected-(U5-DIAG-Pad11) -> VCC
- U5 pad 12: unconnected-(U5-INDEX-Pad12) -> Net-(U5-AVREF)
- U5 pad 13: GND -> Net-(U5-AVREF)
- U5 pad 14: +3.3V -> GND
- U5 pad 15: +3.3V -> +3V3
- U5 pad 16: Net-(U5-STEP) -> unconnected-(U5-NRESET-Pad16)
- U5 pad 17: Net-(U5-VREF) -> unconnected-(U5-NSLEEP-Pad17)
- U5 pad 18: GND -> unconnected-(U5-NFAULT-Pad18)
- U5 pad 19: Net-(U5-DIR) -> unconnected-(U5-DECAY-Pad19)
- U5 pad 2: Net-(U5-ENN) -> Net-(U5-CP2)
- U5 pad 20: GND -> /GPIO9/SPI0.MISO
- U5 pad 21: Net-(J4-Pin_1) -> /GPIO10/SPI0.MOSI
- U5 pad 22: VCC -> /GPIO11/SPI0.SCLK
- U5 pad 23: Net-(U5-BRA) -> unconnected-(U5-NC-Pad23)
- U5 pad 24: Net-(J4-Pin_2) -> Net-(JP7-B)
- U5 pad 25: unconnected-(U5-NC-Pad25) -> Net-(JP8-B)
- U5 pad 26: Net-(J4-Pin_3) -> Net-(JP9-B)
- U5 pad 27: Net-(U5-BRB) -> unconnected-(U5-NHOME-Pad27)
- U5 pad 28: VCC -> GND
- U5 pad 3: GND -> Net-(U5-VCP)
- U5 pad 4: Net-(U5-CPO) -> VCC
- U5 pad 5: Net-(U5-CPI) -> Net-(J3-Pin_2)
- U5 pad 6: Net-(U5-VCP) -> Net-(U5-ISENA)
- U5 pad 7: Net-(JP9-B) -> Net-(J3-Pin_1)
- U5 pad 8: Net-(U5-5VOUT) -> Net-(J3-Pin_4)
- U5 pad 9: Net-(JP7-B) -> Net-(U5-ISENB)
- U6 pad 1: Net-(J5-Pin_4) -> Net-(U6-CP1)
- U6 pad 10: Net-(JP11-B) -> Net-(J5-Pin_3)
- U6 pad 11: unconnected-(U6-DIAG-Pad11) -> VCC
- U6 pad 12: unconnected-(U6-INDEX-Pad12) -> Net-(U6-AVREF)
- U6 pad 13: GND -> Net-(U6-AVREF)
- U6 pad 14: +3.3V -> GND
- U6 pad 15: +3.3V -> +3V3
- U6 pad 16: Net-(U6-STEP) -> unconnected-(U6-NRESET-Pad16)
- U6 pad 17: Net-(U6-VREF) -> unconnected-(U6-NSLEEP-Pad17)
- U6 pad 18: GND -> unconnected-(U6-NFAULT-Pad18)
- U6 pad 19: Net-(U6-DIR) -> unconnected-(U6-DECAY-Pad19)
- U6 pad 2: Net-(U6-ENN) -> Net-(U6-CP2)
- U6 pad 20: GND -> /GPIO5
- U6 pad 21: Net-(J5-Pin_1) -> /GPIO13/PWM1
- U6 pad 22: VCC -> /GPIO6
- U6 pad 23: Net-(U6-BRA) -> unconnected-(U6-NC-Pad23)
- U6 pad 24: Net-(J5-Pin_2) -> Net-(JP10-B)
- U6 pad 25: unconnected-(U6-NC-Pad25) -> Net-(JP11-B)
- U6 pad 26: Net-(J5-Pin_3) -> Net-(JP12-B)
- U6 pad 27: Net-(U6-BRB) -> unconnected-(U6-NHOME-Pad27)
- U6 pad 28: VCC -> GND
- U6 pad 3: GND -> Net-(U6-VCP)
- U6 pad 4: Net-(U6-CPO) -> VCC
- U6 pad 5: Net-(U6-CPI) -> Net-(J5-Pin_2)
- U6 pad 6: Net-(U6-VCP) -> Net-(U6-ISENA)
- U6 pad 7: Net-(JP12-B) -> Net-(J5-Pin_1)
- U6 pad 8: Net-(U6-5VOUT) -> Net-(J5-Pin_4)
- U6 pad 9: Net-(JP10-B) -> Net-(U6-ISENB)
- XSTOP1 pad 1: Net-(XSTOP1-Pin_1) -> /Endstops/Stop X
- YSTOP1 pad 1: Net-(YSTOP1-Pin_1) -> /Endstops/Stop Y
- ZSTOP1 pad 1: Net-(ZSTOP1-Pin_1) -> /Endstops/Stop Z
Other:
- board text added: "Extend PCB edge 0.5mm if using SMT header"
- board text removed: "+5V GND PIN"

Commit message: schematic candidate 0
Parts:
- removed R11, R13: 10K 0402, Resistor_SMD:R_0402_1005Metric
- added C38: 0.1μF 0402 50V, Capacitor_SMD:C_0402_1005Metric, F.Cu at (142.5, 203.1)
- added D4: SMBJ33A, Diode_SMD:D_SMB, F.Cu at (62.5, 223.3)
- added D5: S8KC-13, Diode_SMD:D_SMC, F.Cu at (62.6, 213.7)
- added F1: 3A, Fuse:Fuseholder_Littelfuse_Nano2_154x, F.Cu at (118.2, 175.7)
- added F2: 7A, Fuse:Fuseholder_Littelfuse_Nano2_154x, F.Cu at (53.1, 227.3)
- added F3: 1A, Fuse:Fuseholder_Littelfuse_Nano2_154x, F.Cu at (59.4, 196.8)
- added F4: 1A, Fuse:Fuseholder_Littelfuse_Nano2_154x, F.Cu at (183.1, 145.3)
- added JP13: ID_WP, Jumper:SolderJumper-2_P1.3mm_Open_RoundedPad1.0x1.5mm, F.Cu at (145.5, 202.4)
- added RN1: 100R 4x0603, Resistor_SMD:R_Array_Concave_4x0603, F.Cu at (296.6, 164.6)
- added RN2: 100R 4x0603, Resistor_SMD:R_Array_Concave_4x0603, F.Cu at (250.6, 128.3)
- added RN3: 100R 4x0603, Resistor_SMD:R_Array_Concave_4x0603, F.Cu at (341.2, 166.4)
- added RN4: 100R 4x0603, Resistor_SMD:R_Array_Concave_4x0603, F.Cu at (389.0, 168.7)
- added RN5: 100R 4x0603, Resistor_SMD:R_Array_Concave_4x0603, F.Cu at (169.6, 146.1)
- added U7: M24C32-DFMN6TP, Package_SO:SOIC-8_5.275x5.275mm_P1.27mm, F.Cu at (142.8, 206.8)
- ASTOP1, XSTOP1, YSTOP1, ZSTOP1: footprint Connector_JST:JST_XH_B3B-XH-A_1x03_P2.50mm_Vertical -> rephat-parts:S3B-XH-SM4-TB; moved to B.Cu
- D1: footprint Diode_SMD:D_SMA-SMB_Universal_Handsoldering -> Diode_SMD:D_SMB
- J12, J3, J4, J5, J6: footprint Connector_JST:JST_XH_B4B-XH-A_1x04_P2.50mm_Vertical -> rephat-parts:S4B-XH-SM4-TB; moved to B.Cu
- R10, R12: value 10K 0402 -> 3K9 0402
- R14, R15, R16, R17, R18, R19, R20, R3: value R110 2010 0.7W Film -> R100 0603; footprint Resistor_SMD:R_2010_5025Metric -> Resistor_SMD:R_0603_1608Metric
- RV1, RV2, RV3, RV4: value 100K -> 10K
- moved R19 260.3 mm to (376.4, 151.8)
- moved R20 260.3 mm to (376.4, 154.3)
- moved U6 254.5 mm to (395.8, 129.8)
- moved RV4 250.7 mm to (381.6, 152.1)
- moved JP10 249.2 mm to (389.7, 157.4)
- moved JP11 249.2 mm to (389.7, 160.9)
- moved JP12 249.2 mm to (389.7, 164.5)
- moved C31 247.1 mm to (369.3, 163.0)
- moved C32 243.8 mm to (384.5, 172.0)
- moved C33 243.8 mm to (384.5, 174.0)
- moved C34 243.8 mm to (384.5, 176.0)
- moved C35 243.8 mm to (384.5, 177.9)
- moved C36 243.8 mm to (384.5, 179.9)
- moved R17 216.7 mm to (332.8, 144.6)
- moved R18 216.6 mm to (332.8, 147.1)
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Connections:
- ASTOP1 pad 1: /Endstops/Stop A -> Net-(ASTOP1-Pin_1)
- ASTOP1 pad 3: +5V -> Net-(ASTOP1-Pin_3)
- C13 pad 1: /Endstops/Stop X -> Net-(D3A-K3A4)
- C14 pad 1: /Endstops/Stop Y -> Net-(D2B-K1A2)
- C15 pad 1: /Endstops/Stop Z -> Net-(D2A-K3A4)
- C16 pad 1: /Endstops/Stop A -> Net-(ASTOP1-Pin_1)
- C17 pad 1: +3.3V -> +3V3
- C18 pad 1: +3.3V -> +3V3
- C40 pad 1: Net-(D1-A) -> Net-(D1-K)
- D1 pad 1: GND -> Net-(D1-K)
- D1 pad 2: Net-(D1-A) -> GND
- D2 pad 2: +3V3 -> +5V
- D2 pad 5: +3V3 -> +5V
- D3 pad 2: +3V3 -> +5V
- D3 pad 3: Net-(D3B-K1A2) -> Net-(ASTOP1-Pin_1)
- D3 pad 5: +3V3 -> +5V
- J1 pad 2: Net-(D1-A) -> Net-(D1-K)
- J1 pad 4: Net-(D1-A) -> Net-(D1-K)
- J17 pad 2: +5V -> Net-(J17-Pin_2)
- J2 pad 2: VCC -> Net-(D4-A)
- Q1 pad 2: +5V -> Net-(Q1-S)
- Q1 pad 3: Net-(D1-A) -> Net-(D1-K)
- Q2 pad 5: +5V -> Net-(Q1-S)
- Q2 pad 6: Net-(D1-A) -> Net-(D1-K)
- R10 pad 1: /Endstops/Stop X -> +3V3
- R10 pad 2: Net-(D2A-K3A4) -> /ID_SCL
- R12 pad 1: /Endstops/Stop Z -> +3V3
- R12 pad 2: Net-(D3A-K3A4) -> /ID_SDA
- R6 pad 1: /Endstops/Stop X -> Net-(D3A-K3A4)
- R6 pad 2: +3.3V -> GND
- R7 pad 1: /Endstops/Stop Y -> Net-(D2B-K1A2)
- R7 pad 2: +3.3V -> GND
- R8 pad 1: /Endstops/Stop Z -> Net-(D2A-K3A4)
- R8 pad 2: +3.3V -> GND
- R9 pad 1: /Endstops/Stop A -> Net-(ASTOP1-Pin_1)
- R9 pad 2: +3.3V -> GND
- U2 pad 14: +3.3V -> +3V3
- U3 pad 20: /GPIO3/SCL1 -> Net-(RN2-R3.1)
- U3 pad 21: /GPIO4/GPCLK0 -> Net-(RN2-R2.1)
- U3 pad 22: /GPIO2/SDA1 -> Net-(RN2-R1.1)
- U4 pad 20: /GPIO27 -> Net-(RN1-R3.1)
- U4 pad 21: /GPIO17 -> Net-(RN1-R2.1)
- U4 pad 22: /GPIO22 -> Net-(RN1-R1.1)
- U5 pad 20: /GPIO9/SPI0.MISO -> Net-(RN3-R3.1)
- U5 pad 21: /GPIO10/SPI0.MOSI -> Net-(RN3-R2.1)
- U5 pad 22: /GPIO11/SPI0.SCLK -> Net-(RN3-R1.1)
- U6 pad 20: /GPIO5 -> Net-(RN4-R3.1)
- U6 pad 21: /GPIO13/PWM1 -> Net-(RN4-R2.1)
- U6 pad 22: /GPIO6 -> Net-(RN4-R1.1)
- XSTOP1 pad 1: /Endstops/Stop X -> Net-(D2A-K3A4)
- XSTOP1 pad 3: +5V -> Net-(ASTOP1-Pin_3)
- YSTOP1 pad 1: /Endstops/Stop Y -> Net-(D2B-K1A2)
- YSTOP1 pad 3: +5V -> Net-(ASTOP1-Pin_3)
- ZSTOP1 pad 1: /Endstops/Stop Z -> Net-(D3A-K3A4)
- ZSTOP1 pad 3: +5V -> Net-(ASTOP1-Pin_3)

Commit message: schematic finished
Parts:
- removed C36: 0.1μF 0402 50V, Capacitor_SMD:C_0402_1005Metric
- removed D5: S8KC-13, Diode_SMD:D_SMC
- removed F4: 1A, Fuse:Fuseholder_Littelfuse_Nano2_154x
- removed RN5: 100R 4x0603, Resistor_SMD:R_Array_Concave_4x0603
- removed RV4: 10K, Potentiometer_SMD:Potentiometer_Bourns_TC33X_Vertical
- removed U5: DRV8825PWP, Package_SO:HTSSOP-28-1EP_4.4x9.7mm_P0.65mm_EP3.4x9.5mm_ThermalVias
- added JP14: ext_vsel, Jumper:SolderJumper-3_P1.3mm_Bridged12_RoundedPad1.0x1.5mm, F.Cu at (393.3, 177.3)
- added Q3: BSS138, Package_TO_SOT_SMD:SOT-23, F.Cu at (384.1, 168.6)
- added Q4: BSS138, Package_TO_SOT_SMD:SOT-23, F.Cu at (384.1, 173.3)
- added Q5: BSS138, Package_TO_SOT_SMD:SOT-23, F.Cu at (384.1, 177.9)
- added Q6: BSS138, Package_TO_SOT_SMD:SOT-23, F.Cu at (384.0, 182.6)
- added R11: 20K 0402, Resistor_SMD:R_0402_1005Metric, F.Cu at (238.4, 177.4)
- added R13: 200m 2512 >2W 1%, Resistor_SMD:R_2512_6332Metric, F.Cu at (61.3, 184.0)
- added R21: 100K 0402, Resistor_SMD:R_0402_1005Metric, F.Cu at (387.3, 173.4)
- added R22: 100K 0402, Resistor_SMD:R_0402_1005Metric, F.Cu at (387.1, 177.6)
- added R23: 100K 0402, Resistor_SMD:R_0402_1005Metric, F.Cu at (387.1, 182.7)
- added R26: 8K2 0402, Resistor_SMD:R_0402_1005Metric, F.Cu at (239.2, 149.2)
- added R27: 2K7 0402, Resistor_SMD:R_0402_1005Metric, F.Cu at (239.9, 157.4)
- added R28: 200m 2512 >2W 1%, Resistor_SMD:R_2512_6332Metric, F.Cu at (224.6, 178.8)
- added R29: 200m 2512 >2W 1%, Resistor_SMD:R_2512_6332Metric, F.Cu at (224.4, 161.1)
- added R30: 2K7 0402, Resistor_SMD:R_0402_1005Metric, F.Cu at (100.1, 199.2)
- added R31: 2K7 0402, Resistor_SMD:R_0402_1005Metric, F.Cu at (96.1, 140.6)
- added R32: 20K 0402, Resistor_SMD:R_0402_1005Metric, F.Cu at (103.8, 249.7)
- added R33: 200m 2512 >2W 1%, Resistor_SMD:R_2512_6332Metric, F.Cu at (70.1, 255.1)
- added R34: 200m 2512 >2W 1%, Resistor_SMD:R_2512_6332Metric, F.Cu at (70.1, 260.0)
- added R35: 8K2 0402, Resistor_SMD:R_0402_1005Metric, F.Cu at (103.8, 251.7)
- added R36: 2K7 0402, Resistor_SMD:R_0402_1005Metric, F.Cu at (103.8, 253.7)
- added RV5: 10K, Potentiometer_SMD:Potentiometer_Bourns_TC33X_Vertical, F.Cu at (239.9, 153.8)
- ASTOP1, J12, J3, J4, J5, J6, XSTOP1, YSTOP1, ZSTOP1: moved to F.Cu
- C1, C25: value 100μF THT 36V -> 100 pF 0402 50V; footprint Capacitor_THT:C_Radial_D6.3mm_H11.0mm_P2.50mm -> Capacitor_SMD:C_0402_1005Metric
- C10, C17, C26, C7: value 0.1μF 0402 50V -> 0.1 μF 0402 50V
- C11, C27: value 1μF 0603 50V -> 100μF THT 36V; footprint Capacitor_SMD:C_0402_1005Metric -> Capacitor_THT:C_Radial_D6.3mm_H11.0mm_P2.50mm
- C12, C21, C28: value 0.1μF 0402 50V -> 1μF 0603 50V
- C20, C22, C24, C29: value 1μF 0603 50V -> 0.1μF 0402 50V
- C32, C4: value 0.1μF 0402 50V -> 100 pF 0402 50V
- C35: value 1μF 0603 50V -> 1μF 0402 50V
- C6: value 0.1μF 0402 16V -> 0.1μF 0603 16V
- F2: value 7A -> 1812L110 (1.1A); footprint Fuse:Fuseholder_Littelfuse_Nano2_154x -> Fuse:Fuse_1812_4532Metric
- F3: value 1A -> 1812L110 (1.1A); footprint Fuse:Fuseholder_Littelfuse_Nano2_154x -> Fuse:Fuse_1812_4532Metric
- R14, R3: value R100 0603 -> 20K 0402; footprint Resistor_SMD:R_0603_1608Metric -> Resistor_SMD:R_0402_1005Metric
- R15, R16, R17: value R100 0603 -> 200m 2512 >2W 1%; footprint Resistor_SMD:R_0603_1608Metric -> Resistor_SMD:R_2512_6332Metric
- R18, R19: value R100 0603 -> 8K2 0402; footprint Resistor_SMD:R_0603_1608Metric -> Resistor_SMD:R_0402_1005Metric
- R20: value R100 0603 -> 100K 0402; footprint Resistor_SMD:R_0603_1608Metric -> Resistor_SMD:R_0402_1005Metric
- U2: value SN74LVC07APW -> TB67S109AFTG; footprint Package_SO:TSSOP-14-1EP_4.4x5mm_P0.65mm -> Package_DFN_QFN:QFN-48-1EP_7x7mm_P0.5mm_EP5.45x5.45mm_ThermalVias
- U3, U4, U6: value DRV8825PWP -> TB67S109AFTG; footprint Package_SO:HTSSOP-28-1EP_4.4x9.7mm_P0.65mm_EP3.4x9.5mm_ThermalVias -> Package_DFN_QFN:QFN-48-1EP_7x7mm_P0.5mm_EP5.45x5.45mm_ThermalVias
- moved F2 364.3 mm to (367.8, 43.7), turned to 180 degrees
- moved J17 357.9 mm to (365.3, 37.5)
- moved J2 349.4 mm to (344.3, 37.3)
- moved D4 336.3 mm to (346.9, 43.7), turned to 180 degrees
- moved F3 335.5 mm to (394.0, 173.0)
- moved JP7 323.7 mm to (31.7, 248.5)
- moved JP8 323.7 mm to (31.7, 252.1)
- moved JP9 323.7 mm to (31.7, 255.6)
- moved ASTOP1 299.3 mm to (358.2, 169.4), turned to 0 degrees
- moved XSTOP1 299.3 mm to (358.2, 181.4), turned to 0 degrees
- moved YSTOP1 299.3 mm to (358.2, 193.4), turned to 0 degrees
- moved ZSTOP1 299.3 mm to (358.2, 205.4), turned to 0 degrees
- moved R19 279.4 mm to (100.1, 193.3)
- moved RN3 268.4 mm to (89.5, 259.8)
- moved R17 266.5 mm to (66.3, 141.6)
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Connections:
- C1 pad 1: VCC -> Net-(U2-OSCM)
- C10 pad 1: Net-(U4-CP2) -> +5V
- C10 pad 2: Net-(U4-CP1) -> GND
- C13 pad 1: Net-(D3A-K3A4) -> Net-(Q5-D)
- C14 pad 1: Net-(D2B-K1A2) -> Net-(Q4-D)
- C15 pad 1: Net-(D2A-K3A4) -> Net-(Q3-D)
- C17 pad 1: +3V3 -> +5V
- C18 pad 1: +3V3 -> /Motors/Vref A
- C20 pad 1: +3V3 -> /Motors/Vref Y
- C22 pad 1: VCC -> /Motors/Vref X
- C23 pad 1: Net-(U4-VCP) -> VCC
- C23 pad 2: VCC -> GND
- C24 pad 1: +3V3 -> VCC
- C25 pad 1: VCC -> Net-(U4-OSCM)
- C26 pad 1: Net-(U5-CP2) -> +5V
- C26 pad 2: Net-(U5-CP1) -> GND
- C29 pad 1: +3V3 -> /Motors/Vref Z
- C30 pad 1: Net-(U5-VCP) -> VCC
- C30 pad 2: VCC -> GND
- C32 pad 1: Net-(U6-CP2) -> Net-(U6-OSCM)
- C32 pad 2: Net-(U6-CP1) -> GND
- C4 pad 1: Net-(U3-CP2) -> Net-(U3-OSCM)
- C4 pad 2: Net-(U3-CP1) -> GND
- C7 pad 1: Net-(U3-VCP) -> +5V
- C7 pad 2: VCC -> GND
- D2 pad 2: +5V -> +3V3
- D2 pad 3: Net-(D2B-K1A2) -> /GPIO26
- D2 pad 5: +5V -> +3V3
- D2 pad 6: Net-(D2A-K3A4) -> /GPIO19/PCM.FS
- D3 pad 2: +5V -> +3V3
- D3 pad 3: Net-(ASTOP1-Pin_1) -> /GPIO20/PCM.DIN
- D3 pad 5: +5V -> +3V3
- D3 pad 6: Net-(D3A-K3A4) -> /GPIO21/PCM.DOUT
- D4 pad 1: GND -> VCC
- D4 pad 2: Net-(D4-A) -> GND
- F2 pad 1: Net-(D4-A) -> Net-(J17-Pin_2)
- F2 pad 2: VCC -> +5V
- F3 pad 1: Net-(J17-Pin_2) -> Net-(ASTOP1-Pin_3)
- F3 pad 2: +5V -> VBUS
- J2 pad 2: Net-(D4-A) -> VCC
- R14 pad 1: Net-(U3-ISENB) -> Net-(U3-OSCM)
- R14 pad 2: GND -> +5V
- R15 pad 1: Net-(U3-ISENA) -> VCC
- R15 pad 2: GND -> Net-(R15-Pad2)
- R16 pad 1: Net-(U4-ISENA) -> VCC
- R16 pad 2: GND -> Net-(R16-Pad2)
- R17 pad 1: Net-(U5-ISENB) -> VCC
- R17 pad 2: GND -> Net-(R17-Pad2)
- R18 pad 1: Net-(U5-ISENA) -> +5V
- R18 pad 2: GND -> Net-(R18-Pad2)
- R19 pad 1: Net-(U6-ISENB) -> +5V
- R19 pad 2: GND -> Net-(R19-Pad2)
- R20 pad 1: Net-(U6-ISENA) -> +3V3
- R20 pad 2: GND -> /GPIO19/PCM.FS
- R3 pad 1: Net-(U4-ISENB) -> Net-(U2-OSCM)
- R3 pad 2: GND -> +5V
- R6 pad 1: Net-(D3A-K3A4) -> Net-(ASTOP1-Pin_3)
- R6 pad 2: GND -> Net-(Q5-D)
- R7 pad 1: Net-(D2B-K1A2) -> Net-(ASTOP1-Pin_3)
- R7 pad 2: GND -> Net-(Q4-D)
- R8 pad 1: Net-(D2A-K3A4) -> Net-(ASTOP1-Pin_3)
- R8 pad 2: GND -> Net-(Q3-D)
- R9 pad 1: Net-(ASTOP1-Pin_1) -> Net-(ASTOP1-Pin_3)
- R9 pad 2: GND -> Net-(ASTOP1-Pin_1)
- RN4 pad 6: /GPIO5 -> /GPIO6
- RN4 pad 7: /GPIO13/PWM1 -> /GPIO5
- RN4 pad 8: /GPIO6 -> /GPIO13/PWM1
- RV1 pad 1: +3V3 -> Net-(R18-Pad2)
- RV1 pad 2: Net-(U3-AVREF) -> /Motors/Vref X
- RV1 pad 3: GND -> Net-(R31-Pad1)
- RV2 pad 1: +3V3 -> Net-(R19-Pad2)
- RV2 pad 2: Net-(U4-AVREF) -> /Motors/Vref Y
- RV2 pad 3: GND -> Net-(R30-Pad1)
- RV3 pad 1: +3V3 -> Net-(R35-Pad2)
- RV3 pad 2: Net-(U5-AVREF) -> /Motors/Vref Z
- RV3 pad 3: GND -> Net-(R36-Pad1)
- U2 pad 1: /Endstops/Stop X -> unconnected-(U2-NC-Pad1)
- U2 pad 10: unconnected-(U2-5Y-Pad10) -> Net-(J4-Pin_2)
- U2 pad 11: unconnected-(U2-5A-Pad11) -> Net-(J4-Pin_2)
- U2 pad 14: +3V3 -> unconnected-(U2-NC-Pad14)
- U2 pad 15: (no net) -> GND
- U2 pad 2: /GPIO19/PCM.FS -> Net-(RN1-R3.1)
- U2 pad 3: /Endstops/Stop Y -> Net-(RN1-R1.1)
- U2 pad 4: /GPIO26 -> GND
- U2 pad 5: /Endstops/Stop Z -> GND
- U2 pad 6: /GPIO21/PCM.DOUT -> unconnected-(U2-NC-Pad6)
- U2 pad 7: GND -> Net-(R13-Pad2)
- U2 pad 8: /GPIO20/PCM.DIN -> Net-(R13-Pad2)
- U2 pad 9: /Endstops/Stop A -> unconnected-(U2-NC-Pad9)
- U3 pad 1: Net-(U3-CP1) -> unconnected-(U3-NC-Pad1)
- U3 pad 10: Net-(J12-Pin_3) -> Net-(J12-Pin_2)
- U3 pad 11: VCC -> Net-(J12-Pin_2)
- U3 pad 12: Net-(U3-AVREF) -> unconnected-(U3-NC-Pad12)
- U3 pad 13: Net-(U3-AVREF) -> unconnected-(U3-NC-Pad13)
- U3 pad 14: GND -> unconnected-(U3-NC-Pad14)
- U3 pad 15: +3V3 -> GND
- U3 pad 16: unconnected-(U3-NRESET-Pad16) -> Net-(J12-Pin_1)
- U3 pad 17: unconnected-(U3-NSLEEP-Pad17) -> Net-(J12-Pin_1)
- U3 pad 18: unconnected-(U3-NFAULT-Pad18) -> GND
- U3 pad 19: unconnected-(U3-DECAY-Pad19) -> GND
- U3 pad 2: Net-(U3-CP2) -> Net-(RN2-R3.1)
- U3 pad 20: Net-(RN2-R3.1) -> Net-(J12-Pin_4)
- U3 pad 21: Net-(RN2-R2.1) -> Net-(J12-Pin_4)
- U3 pad 22: Net-(RN2-R1.1) -> GND
- U3 pad 24: Net-(JP1-B) -> unconnected-(U3-NC-Pad24)
- U3 pad 25: Net-(JP2-B) -> unconnected-(U3-NC-Pad25)
- U3 pad 26: Net-(JP3-B) -> Net-(J12-Pin_3)
- U3 pad 27: unconnected-(U3-NHOME-Pad27) -> Net-(J12-Pin_3)
- U3 pad 28: GND -> unconnected-(U3-NC-Pad28)
- U3 pad 29: GND -> Net-(R17-Pad2)
- U3 pad 3: Net-(U3-VCP) -> Net-(RN2-R1.1)
- U3 pad 4: VCC -> GND
- U3 pad 5: Net-(J12-Pin_2) -> GND
- U3 pad 6: Net-(U3-ISENA) -> unconnected-(U3-NC-Pad6)
- U3 pad 7: Net-(J12-Pin_1) -> Net-(R15-Pad2)
- U3 pad 8: Net-(J12-Pin_4) -> Net-(R15-Pad2)
- U3 pad 9: Net-(U3-ISENB) -> unconnected-(U3-NC-Pad9)
- U4 pad 1: Net-(U4-CP1) -> unconnected-(U4-NC-Pad1)
- U4 pad 10: Net-(J4-Pin_3) -> Net-(J3-Pin_2)
- U4 pad 11: VCC -> Net-(J3-Pin_2)
- U4 pad 12: Net-(U4-AVREF) -> unconnected-(U4-NC-Pad12)
- U4 pad 13: Net-(U4-AVREF) -> unconnected-(U4-NC-Pad13)
- U4 pad 14: GND -> unconnected-(U4-NC-Pad14)
- U4 pad 15: +3V3 -> GND
- U4 pad 16: unconnected-(U4-NRESET-Pad16) -> Net-(J3-Pin_1)
- U4 pad 17: unconnected-(U4-NSLEEP-Pad17) -> Net-(J3-Pin_1)
- U4 pad 18: unconnected-(U4-NFAULT-Pad18) -> GND
- U4 pad 19: unconnected-(U4-DECAY-Pad19) -> GND
- U4 pad 2: Net-(U4-CP2) -> Net-(RN3-R3.1)
- U4 pad 20: Net-(RN1-R3.1) -> Net-(J3-Pin_4)
- U4 pad 21: Net-(RN1-R2.1) -> Net-(J3-Pin_4)
- U4 pad 22: Net-(RN1-R1.1) -> GND
- U4 pad 24: Net-(JP4-B) -> unconnected-(U4-NC-Pad24)
- U4 pad 25: Net-(JP5-B) -> unconnected-(U4-NC-Pad25)
- U4 pad 26: Net-(JP6-B) -> Net-(J3-Pin_3)
- U4 pad 27: unconnected-(U4-NHOME-Pad27) -> Net-(J3-Pin_3)
- U4 pad 28: GND -> unconnected-(U4-NC-Pad28)
- U4 pad 29: GND -> Net-(R34-Pad2)
- U4 pad 3: Net-(U4-VCP) -> Net-(RN3-R1.1)
- U4 pad 4: VCC -> GND
- U4 pad 5: Net-(J4-Pin_2) -> GND
- U4 pad 6: Net-(U4-ISENA) -> unconnected-(U4-NC-Pad6)
- U4 pad 7: Net-(J4-Pin_1) -> Net-(R33-Pad2)
- U4 pad 8: Net-(J4-Pin_4) -> Net-(R33-Pad2)
- U4 pad 9: Net-(U4-ISENB) -> unconnected-(U4-NC-Pad9)
- U6 pad 1: Net-(U6-CP1) -> unconnected-(U6-NC-Pad1)
- U6 pad 10: Net-(J5-Pin_3) -> Net-(J5-Pin_2)
- U6 pad 11: VCC -> Net-(J5-Pin_2)
- U6 pad 12: Net-(U6-AVREF) -> unconnected-(U6-NC-Pad12)
- U6 pad 13: Net-(U6-AVREF) -> unconnected-(U6-NC-Pad13)
- U6 pad 14: GND -> unconnected-(U6-NC-Pad14)
- U6 pad 15: +3V3 -> GND
- U6 pad 16: unconnected-(U6-NRESET-Pad16) -> Net-(J5-Pin_1)
- U6 pad 17: unconnected-(U6-NSLEEP-Pad17) -> Net-(J5-Pin_1)
- U6 pad 18: unconnected-(U6-NFAULT-Pad18) -> GND
- U6 pad 19: unconnected-(U6-DECAY-Pad19) -> GND
- U6 pad 2: Net-(U6-CP2) -> Net-(RN4-R3.1)
- U6 pad 20: Net-(RN4-R3.1) -> Net-(J5-Pin_4)
- U6 pad 21: Net-(RN4-R2.1) -> Net-(J5-Pin_4)
- U6 pad 22: Net-(RN4-R1.1) -> GND
- U6 pad 24: Net-(JP10-B) -> unconnected-(U6-NC-Pad24)
- U6 pad 25: Net-(JP11-B) -> unconnected-(U6-NC-Pad25)
- U6 pad 26: Net-(JP12-B) -> Net-(J5-Pin_3)
- U6 pad 27: unconnected-(U6-NHOME-Pad27) -> Net-(J5-Pin_3)
- U6 pad 28: GND -> unconnected-(U6-NC-Pad28)
- U6 pad 29: GND -> Net-(R29-Pad2)
- U6 pad 3: Net-(U6-VCP) -> Net-(RN4-R1.1)
- U6 pad 4: VCC -> GND
- U6 pad 5: Net-(J5-Pin_2) -> GND
- U6 pad 6: Net-(U6-ISENA) -> unconnected-(U6-NC-Pad6)
- U6 pad 7: Net-(J5-Pin_1) -> Net-(R28-Pad2)
- U6 pad 8: Net-(J5-Pin_4) -> Net-(R28-Pad2)
- U6 pad 9: Net-(U6-ISENB) -> unconnected-(U6-NC-Pad9)
- XSTOP1 pad 1: Net-(D2A-K3A4) -> Net-(Q3-D)
- YSTOP1 pad 1: Net-(D2B-K1A2) -> Net-(Q4-D)
- ZSTOP1 pad 1: Net-(D3A-K3A4) -> Net-(Q5-D)
