File: kicad/RepHat.kicad_pcb (KiCad board)
At the start: 2 copper layers, 65 x 56 mm, 132 parts, among them J1 GPIO, J12 Conn_01x04_Pin, J13 Conn_01x03_Pin, J17 Screw_Terminal_01x02, J2 Screw_Terminal_01x02, J3 Conn_01x04_Pin, J4 Conn_01x04_Pin, J5 Conn_01x04_Pin, J6 Conn_01x04_Pin, Q1 DMG2301L, Q2 DMMT5401, Q3 BSS138, Q4 BSS138, Q5 BSS138, Q6 BSS138, U1 LMR51450FNDRRR, U2 TB67S109AFTG, U3 TB67S109AFTG, U4 TB67S109AFTG, U6 TB67S109AFTG, U7 M24C32-DFMN6TP

Commit message: layout progress
Parts:
- moved RN3 212.2 mm to (133.8, 52.2), turned to 90 degrees
- moved RN1 158.9 mm to (123.6, 52.4), turned to 90 degrees
- moved R5 144.3 mm to (243.0, 86.0), turned to -90 degrees
- moved L1 142.6 mm to (239.1, 76.2), turned to -160 degrees
- moved C13 142.3 mm to (249.6, 123.3)
- moved C14 142.3 mm to (249.6, 118.6)
- moved C15 142.3 mm to (249.6, 114.0)
- moved JP14 142.3 mm to (261.5, 123.6)
- moved R6 142.3 mm to (249.6, 125.3)
- moved R7 142.3 mm to (249.6, 120.7)
- moved R8 142.3 mm to (249.6, 116.1)
- moved C16 142.3 mm to (249.5, 127.9)
- moved D2 142.3 mm to (256.0, 117.2)
- moved Q3 142.3 mm to (252.2, 115.0)
- moved Q4 142.3 mm to (252.2, 119.6)
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Connections:
- U2 pad 10: Net-(J4-Pin_2) -> Net-(J4-Pin_1)
- U2 pad 11: Net-(J4-Pin_2) -> Net-(J4-Pin_1)
- U2 pad 16: Net-(J4-Pin_1) -> Net-(J4-Pin_2)
- U2 pad 17: Net-(J4-Pin_1) -> Net-(J4-Pin_2)
- U2 pad 20: Net-(J4-Pin_4) -> Net-(J4-Pin_3)
- U2 pad 21: Net-(J4-Pin_4) -> Net-(J4-Pin_3)
- U2 pad 26: Net-(J4-Pin_3) -> Net-(J4-Pin_4)
- U2 pad 27: Net-(J4-Pin_3) -> Net-(J4-Pin_4)
- U2 pad 49: (no net) -> GND
- U3 pad 10: Net-(J12-Pin_2) -> Net-(J12-Pin_1)
- U3 pad 11: Net-(J12-Pin_2) -> Net-(J12-Pin_1)
- U3 pad 16: Net-(J12-Pin_1) -> Net-(J12-Pin_2)
- U3 pad 17: Net-(J12-Pin_1) -> Net-(J12-Pin_2)
- U3 pad 20: Net-(J12-Pin_4) -> Net-(J12-Pin_3)
- U3 pad 21: Net-(J12-Pin_4) -> Net-(J12-Pin_3)
- U3 pad 26: Net-(J12-Pin_3) -> Net-(J12-Pin_4)
- U3 pad 27: Net-(J12-Pin_3) -> Net-(J12-Pin_4)
- U3 pad 49: (no net) -> GND
- U4 pad 10: Net-(J3-Pin_2) -> Net-(J3-Pin_1)
- U4 pad 11: Net-(J3-Pin_2) -> Net-(J3-Pin_1)
- U4 pad 16: Net-(J3-Pin_1) -> Net-(J3-Pin_2)
- U4 pad 17: Net-(J3-Pin_1) -> Net-(J3-Pin_2)
- U4 pad 20: Net-(J3-Pin_4) -> Net-(J3-Pin_3)
- U4 pad 21: Net-(J3-Pin_4) -> Net-(J3-Pin_3)
- U4 pad 26: Net-(J3-Pin_3) -> Net-(J3-Pin_4)
- U4 pad 27: Net-(J3-Pin_3) -> Net-(J3-Pin_4)
- U4 pad 49: (no net) -> GND
- U6 pad 10: Net-(J5-Pin_2) -> Net-(J5-Pin_1)
- U6 pad 11: Net-(J5-Pin_2) -> Net-(J5-Pin_1)
- U6 pad 16: Net-(J5-Pin_1) -> Net-(J5-Pin_2)
- U6 pad 17: Net-(J5-Pin_1) -> Net-(J5-Pin_2)
- U6 pad 20: Net-(J5-Pin_4) -> Net-(J5-Pin_3)
- U6 pad 21: Net-(J5-Pin_4) -> Net-(J5-Pin_3)
- U6 pad 26: Net-(J5-Pin_3) -> Net-(J5-Pin_4)
- U6 pad 27: Net-(J5-Pin_3) -> Net-(J5-Pin_4)
- U6 pad 49: (no net) -> GND
Other:
- outline, holes or cut-outs redrawn
- board text removed: "Extend PCB edge 0.5mm if using SMT header"
